File: MiP D1 mini Pack/MiP D1 mini Pack.kicad_pcb (KiCad board)
At the start: 2 copper layers, 41.4 x 63.8 mm, 12 parts, among them J3 Debug, U1 WEMOS_D1_mini

Commit message: Schematic cleanup
Renamed the connector references to account for the lost J1 and J2 from the v2 board.  Moved things around a bit.
Parts:
- U1: value WEMOS_D1_mini -> WEMOS D1 mini
- renumbered JP11 to J1, J3 to J2
Changed lines of the file:
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@@
 		(descr "Through hole angled socket strip, 1x02, 2.54mm pitch, 8.51mm socket length, single row (from Kicad 4.0.7), script generated")
 		(tags "Through hole angled socket strip THT 1x02 2.54mm single row")
-		(property "Reference" "J3"
+		(property "Reference" "J2"
 			(at -4.38 -2.77 90)
 			(layer "F.SilkS")
@@
 			)
 		)
-		(property "Value" "WEMOS_D1_mini"
+		(property "Value" "WEMOS D1 mini"
 			(at 11.7 0 0)
 			(layer "F.Fab")
@@
 		(descr "JST ZH series connector, B4B-ZR (http://www.jst-mfg.com/product/pdf/eng/eZH.pdf)")
 		(tags "connector JST ZH vertical")
-		(property "Reference" "JP11"
+		(property "Reference" "J1"
 			(at 2.25 2.5 90)
 			(layer "B.SilkS")
